File: ft232.sch (EAGLE design)
At the start: 12 parts, among them U1 FT232RL-BASICSSOP

Commit message: Added CAM files
Connections:
- net GND: now also JP1.GND
Changed lines of the file:
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@@
 <part name="GND4" library="supply1" deviceset="GND" device=""/>
 <part name="GND5" library="supply1" deviceset="GND" device=""/>
+<part name="GND6" library="supply1" deviceset="GND" device=""/>
 </parts>
 <sheets>
@@
 <instance part="GND4" gate="1" x="22.86" y="91.44"/>
 <instance part="GND5" gate="1" x="76.2" y="91.44"/>
+<instance part="GND6" gate="1" x="17.78" y="114.3"/>
 </instances>
 <busses>
@@
 <label x="88.9" y="71.12" size="1.778" layer="95"/>
 </segment>
+<segment>
+<pinref part="JP1" gate="G$1" pin="GND"/>
+<pinref part="GND6" gate="1" pin="GND"/>
+<wire x1="15.24" y1="119.38" x2="17.78" y2="119.38" width="0.1524" layer="91"/>
+<wire x1="17.78" y1="119.38" x2="17.78" y2="116.84" width="0.1524" layer="91"/>
+</segment>
 </net>
